File: relay-prototype/page1.kicad_sch (KiCad schematic)
At the start: 28 parts, among them K1 G5V-1, K10 G5V-1, K11 G5V-1, K12 G5V-1, K13 G5V-1, K14 G5V-1, K2 G5V-1, K3 G5V-1, K4 G5V-1, K5 G5V-1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

Commit message: prototype board completed, usb 3d model added
Parts:
- D1: footprint Diode_THT:D_DO-15_P12.70mm_Horizontal -> Diode_SMD:D_SOD-323_HandSoldering; Part_Link (none) -> https://www.digikey.com/short/zpm0qwdt
- D10, D11, D12, D13, D14, D2, D3, D4, D5, D6, D7, D8, D9: footprint Diode_THT:D_DO-15_P12.70mm_Horizontal -> Diode_SMD:D_SOD-323_HandSoldering
Changed lines of the file:
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@@
       (effects (font (size 1.27 1.27)) (justify right) hide)
     )
-    (property "Footprint" "Diode_THT:D_DO-15_P12.70mm_Horizontal" (at 34.29 132.08 0)
+    (property "Footprint" "Diode_SMD:D_SOD-323_HandSoldering" (at 34.29 132.08 0)
       (effects (font (size 1.27 1.27)) hide)
     )
@@
       (effects (font (size 1.27 1.27)) (justify right) hide)
     )
-    (property "Footprint" "Diode_THT:D_DO-15_P12.70mm_Horizontal" (at 72.39 134.62 0)
+    (property "Footprint" "Diode_SMD:D_SOD-323_HandSoldering" (at 72.39 134.62 0)
       (effects (font (size 1.27 1.27)) hide)
     )
@@
       (effects (font (size 1.27 1.27)) (justify right) hide)
     )
-    (property "Footprint" "Diode_THT:D_DO-15_P12.70mm_Horizontal" (at 73.66 77.47 0)
+    (property "Footprint" "Diode_SMD:D_SOD-323_HandSoldering" (at 73.66 77.47 0)
       (effects (font (size 1.27 1.27)) hide)
     )
@@
       (effects (font (size 1.27 1.27)) (justify right) hide)
     )
-    (property "Footprint" "Diode_THT:D_DO-15_P12.70mm_Horizontal" (at 172.72 130.81 0)
+    (property "Footprint" "Diode_SMD:D_SOD-323_HandSoldering" (at 172.72 130.81 0)
       (effects (font (size 1.27 1.27)) hide)
     )
@@
       (effects (font (size 1.27 1.27)) (justify right) hide)
     )
-    (property "Footprint" "Diode_THT:D_DO-15_P12.70mm_Horizontal" (at 36.83 46.99 0)
+    (property "Footprint" "Diode_SMD:D_SOD-323_HandSoldering" (at 36.83 46.99 0)
       (effects (font (size 1.27 1.27)) hide)
     )
@@
       (effects (font (size 1.27 1.27)) hide)
     )
+    (property "Part_Link" "https://www.digikey.com/short/zpm0qwdt" (at 36.83 46.99 90)
+      (effects (font (size 1.27 1.27)) hide)
+    )
     (pin "1")
     (pin "2")
@@
       (effects (font (size 1.27 1.27)) (justify right) hide)
     )
-    (property "Footprint" "Diode_THT:D_DO-15_P12.70mm_Horizontal" (at 172.72 74.93 0)
+    (property "Footprint" "Diode_SMD:D_SOD-323_HandSoldering" (at 172.72 74.93 0)
       (effects (font (size 1.27 1.27)) hide)
     )
@@
       (effects (font (size 1.27 1.27)) (justify right) hide)
     )
-    (property "Footprint" "Diode_THT:D_DO-15_P12.70mm_Horizontal" (at 172.72 46.99 0)
+    (property "Footprint" "Diode_SMD:D_SOD-323_HandSoldering" (at 172.72 46.99 0)
       (effects (font (size 1.27 1.27)) hide)
     )
@@
       (effects (font (size 1.27 1.27)) (justify right) hide)
     )
-    (property "Footprint" "Diode_THT:D_DO-15_P12.70mm_Horizontal" (at 172.72 102.87 0)
+    (property "Footprint" "Diode_SMD:D_SOD-323_HandSoldering" (at 172.72 102.87 0)
       (effects (font (size 1.27 1.27)) hide)
     )
@@
       (effects (font (size 1.27 1.27)) (justify right) hide)
     )
-    (property "Footprint" "Diode_THT:D_DO-15_P12.70mm_Horizontal" (at 100.33 77.47 0)
+    (property "Footprint" "Diode_SMD:D_SOD-323_HandSoldering" (at 100.33 77.47 0)
       (effects (font (size 1.27 1.27)) hide)
     )
@@
       (effects (font (size 1.27 1.27)) (justify right) hide)
     )
-    (property "Footprint" "Diode_THT:D_DO-15_P12.70mm_Horizontal" (at 35.56 74.93 0)
+    (property "Footprint" "Diode_SMD:D_SOD-323_HandSoldering" (at 35.56 74.93 0)
       (effects (font (size 1.27 1.27)) hide)
     )
@@
       (effects (font (size 1.27 1.27)) (justify right) hide)
     )
-    (property "Footprint" "Diode_THT:D_DO-15_P12.70mm_Horizontal" (at 66.04 110.49 0)
+    (property "Footprint" "Diode_SMD:D_SOD-323_HandSoldering" (at 66.04 110.49 0)
       (effects (font (size 1.27 1.27)) hide)
     )
@@
       (effects (font (size 1.27 1.27)) (justify right) hide)
     )
-    (property "Footprint" "Diode_THT:D_DO-15_P12.70mm_Horizontal" (at 99.06 134.62 0)
+    (property "Footprint" "Diode_SMD:D_SOD-323_HandSoldering" (at 99.06 134.62 0)
       (effects (font (size 1.27 1.27)) hide)
     )
@@
       (effects (font (size 1.27 1.27)) (justify right) hide)
     )
-    (property "Footprint" "Diode_THT:D_DO-15_P12.70mm_Horizontal" (at 35.56 104.14 0)
+    (property "Footprint" "Diode_SMD:D_SOD-323_HandSoldering" (at 35.56 104.14 0)
       (effects (font (size 1.27 1.27)) hide)
     )
@@
       (effects (font (size 1.27 1.27)) (justify right) hide)
     )
-    (property "Footprint" "Diode_THT:D_DO-15_P12.70mm_Horizontal" (at 67.31 53.34 0)
-      (effects (font (size 1.27 1.27)) hide)
-    )
+    (property "Footprint" "Diode_SMD:D_SOD-323_HandSoldering" (at 67.31 53.34 0)
+      (effects (font (size 1.27 1.27)) hide)
+    )
