File: relay-prototype/page2.kicad_sch (KiCad schematic)
At the start: 8 parts, among them K1 G5V-1

Commit message: start of pcb, usb-c connector
Parts:
- LED4: footprint (none) -> LED_THT:LED_D5.0mm
Changed lines of the file:
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@@
       (effects (font (size 1.27 1.27)) hide)
     )
-    (property "Footprint" "" (at 115.57 38.1 0)
+    (property "Footprint" "LED_THT:LED_D5.0mm" (at 115.57 38.1 0)
       (effects (font (size 1.27 1.27)) hide)
     )
@@
       (effects (font (size 1.27 1.27)) hide)
     )
-    (property "Footprint" "" (at 115.57 30.48 0)
+    (property "Footprint" "LED_THT:LED_D5.0mm" (at 115.57 30.48 0)
       (effects (font (size 1.27 1.27)) hide)
     )

Commit message: prototype board completed, usb 3d model added
Parts:
- D1: footprint Diode_THT:D_DO-15_P12.70mm_Horizontal -> Diode_SMD:D_SOD-323_HandSoldering
- R8: value 300 -> 330
Changed lines of the file:
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@@
       (effects (font (size 1.27 1.27)))
     )
-    (property "Value" "300" (at 106.68 30.48 90)
+    (property "Value" "330" (at 106.68 30.48 90)
       (effects (font (size 1.27 1.27)))
     )
@@
       (effects (font (size 1.27 1.27)) (justify right) hide)
     )
-    (property "Footprint" "Diode_THT:D_DO-15_P12.70mm_Horizontal" (at 44.45 67.31 0)
+    (property "Footprint" "Diode_SMD:D_SOD-323_HandSoldering" (at 44.45 67.31 0)
       (effects (font (size 1.27 1.27)) hide)
     )
@@
       (effects (font (size 1.27 1.27)) (justify right) hide)
     )
-    (property "Footprint" "Diode_THT:D_DO-15_P12.70mm_Horizontal" (at 44.45 39.37 0)
+    (property "Footprint" "Diode_SMD:D_SOD-323_HandSoldering" (at 44.45 39.37 0)
       (effects (font (size 1.27 1.27)) hide)
     )
@@
       (effects (font (size 1.27 1.27)))
     )
-    (property "Value" "300" (at 106.68 38.1 90)
-      (effects (font (size 1.27 1.27)))
-    )
+    (property "Value" "330" (at 106.68 38.1 90)
+      (effects (font (size 1.27 1.27)))
+    )
