File: relay-prototype/relay-prototype.kicad_pcb (KiCad board)
At the start: 2 copper layers, 64 parts, among them K1 G5V-1, K10 G5V-1, K11 G5V-1, K12 G5V-1, K13 G5V-1, K14 G5V-1, K15 G5V-1, K16 G5V-1, K17 G5V-1, K18 G5V-1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

Commit message: start of pcb, usb-c connector
Parts:
- added J1: USB_C_Receptacle_PowerOnly_6P, USB-C-Power-tester:TYPE-C-31-M-17_handsolder, F.Cu at (264.2, 116.8)
- added RCC1: 5.1K, Resistor_THT:R_Axial_DIN0207_L6.3mm_D2.5mm_P10.16mm_Horizontal, F.Cu at (260.4, 104.9)
- added RCC2: 5.1K, Resistor_THT:R_Axial_DIN0207_L6.3mm_D2.5mm_P10.16mm_Horizontal, F.Cu at (260.4, 108.9)
- R1, R10, R11, R2, R3, R4, R5, R6, R7, R8: moved to B.Cu
- moved D21 153.1 mm to (288.7, 130.8)
- moved K21 150.8 mm to (296.1, 108.3)
- moved D1 150.8 mm to (222.5, 56.3)
- moved D10 150.8 mm to (222.5, 102.7)
- moved D11 150.8 mm to (222.5, 107.8)
- moved D12 150.8 mm to (222.5, 113.0)
- moved D13 150.8 mm to (222.5, 118.1)
- moved D14 150.8 mm to (222.5, 123.3)
- moved D2 150.8 mm to (222.5, 61.5)
- moved D3 150.8 mm to (222.5, 66.6)
- moved D4 150.8 mm to (222.5, 71.8)
- moved D5 150.8 mm to (222.5, 76.9)
- moved D6 150.8 mm to (222.5, 82.1)
- moved D7 150.8 mm to (222.5, 87.2)
- moved D8 150.8 mm to (222.5, 92.4)
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
Commit message: prototype board completed, usb 3d model added
Parts:
- D1, D10, D11, D12, D13, D14, D15, D16, D17, D18, D19, D2, D20, D21, D3, D4, D5, D6, D7, D8, D9: footprint Diode_THT:D_DO-15_P12.70mm_Horizontal -> Diode_SMD:D_SOD-323_HandSoldering; moved to B.Cu
- R10, R11, R5, R6, R7, R8: value 300 -> 330
- R9, RCC1, RCC2: moved to B.Cu
- moved R9 210.2 mm to (76.3, 108.9), turned to 90 degrees
- moved K5 180.6 mm to (95.3, 51.1), turned to 90 degrees
- moved K20 175.4 mm to (111.7, 101.9), turned to 90 degrees
- moved D20 171.7 mm to (116.7, 99.5), turned to 90 degrees
- moved K4 171.4 mm to (95.3, 61.3), turned to 90 degrees
- moved J1 168.1 mm to (96.1, 111.3)
- moved K21 168.0 mm to (128.2, 101.9), turned to 90 degrees
- moved K10 165.0 mm to (111.9, 51.1), turned to 90 degrees
- moved K3 163.0 mm to (95.3, 71.4), turned to 90 degrees
- moved D21 158.6 mm to (133.2, 99.5), turned to 90 degrees
- moved K2 155.2 mm to (95.3, 81.6), turned to 90 degrees
- moved K9 155.1 mm to (111.9, 61.3), turned to 90 degrees
- moved K8 145.7 mm to (111.9, 71.4), turned to 90 degrees
- moved K14 142.1 mm to (128.5, 51.0), turned to 90 degrees
- moved RCC1 137.2 mm to (123.3, 110.2), turned to 180 degrees
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Routing:
- net A1: track 0.00 -> 218.2 mm, vias 0 -> 2
- net A0: track 0.00 -> 119.2 mm
- net CIN0: track 0.00 -> 101.8 mm
- net OUT1: track 0.00 -> 92.5 mm
- net ADDCOUT0: track 0.00 -> 86.7 mm
- net Net-(D7-A2): track 0.00 -> 82.7 mm
- net Net-(D19-A2): track 0.00 -> 81.6 mm
- net B1: track 0.00 -> 80.0 mm
- net Net-(D2-A2): track 0.00 -> 68.3 mm
- net B0: track 0.00 -> 67.2 mm
- net OUT0: track 0.00 -> 60.1 mm
- net SELECT: track 0.00 -> 59.9 mm
- net SUB0: track 0.00 -> 58.0 mm
- net GND: track 0.00 -> 55.8 mm, vias 0 -> 2
- net SUB1: track 0.00 -> 52.6 mm
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- added copper zone on In1.Cu, net +5V
- added copper zone on In2.Cu, net GND
Other:
- board outline added: 91.4 x 71.1 mm
- copper layers 2 -> 4
- board text added: "0"
- board text added: "1"
- board text added: "ADD"
- board text added: "INPUT"
- board text added: "OUTPUT"
- board text added: "SUB"
